Commit message: updated gazebo launch file

File: ijamul_description/urdf/ijamul.urdf.xacro (robot description, xacro)
@@ -47,5 +47,5 @@
     <origin xyz="0 0 0.007" rpy="0 0 0"/>
   </joint>
-  <link name="wheel_right_link">
+  <link name="wheel_left_link">
     <inertial>
       <origin xyz="0 0.014 0" rpy="0 0 0" />
@@ -69,5 +69,5 @@
     </collision>
   </link>
-   <joint name="wheel_right_joint" type="continuous">
+   <joint name="wheel_left_joint" type="continuous">
     <origin xyz="0.0312 -0.09764 -0.003" rpy="0 0 0" />
     <parent link="base_link" />
@@ -76,5 +76,5 @@
   </joint>
   <link
-    name="wheel_left_link">
+    name="wheel_right_link">
     <inertial>
       <origin xyz="0 0.014 0" rpy="0 0 0" />
@@ -98,5 +98,5 @@
     </collision>
   </link>
-  <joint name="wheel_left_joint" type="continuous">
+  <joint name="wheel_right_joint" type="continuous">
     <origin xyz="0.0312 0.09764 -0.003" rpy="0 0 0" />
     <parent link="base_link" />

Commit message: included localization and navigation data

File: ijamul_description/urdf/ijamul.urdf.xacro (robot description, xacro)
@@ -8,4 +8,8 @@
   <xacro:include filename="$(find ijamul_description)/urdf/ijamul_ros2_control.xacro" />
   <xacro:include filename="$(find ijamul_description)/urdf/inertial_macros.xacro"/>
+  <!-- Include Gazebo Parameters -->
+  <xacro:include filename="$(find ijamul_description)/urdf/imu.urdf.xacro" />
+  <!-- Include Gazebo Parameters -->
+  <xacro:include filename="$(find ijamul_description)/urdf/generic_laser.urdf.xacro" />
   <xacro:property name="caster_wheel_radius" value="0.03"/>
   <xacro:property name="caster_wheel_mass" value="0.01"/>
@@ -47,5 +51,5 @@
     <origin xyz="0 0 0.007" rpy="0 0 0"/>
   </joint>
-  <link name="wheel_left_link">
+  <link name="wheel_right_link">
     <inertial>
       <origin xyz="0 0.014 0" rpy="0 0 0" />
@@ -69,5 +73,5 @@
     </collision>
   </link>
-   <joint name="wheel_left_joint" type="continuous">
+   <joint name="wheel_right_joint" type="continuous">
     <origin xyz="0.0312 -0.09764 -0.003" rpy="0 0 0" />
     <parent link="base_link" />
@@ -76,5 +80,5 @@
   </joint>
   <link
-    name="wheel_right_link">
+    name="wheel_left_link">
     <inertial>
       <origin xyz="0 0.014 0" rpy="0 0 0" />
@@ -98,5 +102,5 @@
     </collision>
   </link>
-  <joint name="wheel_right_joint" type="continuous">
+  <joint name="wheel_left_joint" type="continuous">
     <origin xyz="0.0312 0.09764 -0.003" rpy="0 0 0" />
     <parent link="base_link" />
@@ -126,3 +130,7 @@
     <axis xyz="0 0 0" />
   </joint>
+  <xacro:imu/>
+  <xacro:generic_laser>
+    <origin xyz="0.06 0 0.05" rpy="0 0 0"/>
+  </xacro:generic_laser>
 </robot>

Commit message: updated display.launch

File: ijamul_description/urdf/ijamul.urdf.xacro (robot description, xacro)
@@ -35,5 +35,5 @@
       <origin xyz="0 0 0" rpy="0 0 0" />
       <geometry>
-        <box size="0.219 0.214 0.06"/>
+        <box size="0.219 0.18 0.06"/>
       </geometry>
       <material name="black"/>
@@ -42,5 +42,5 @@
       <origin xyz="0 0 0" rpy="0 0 0" />
       <geometry>
-        <box size="0.219 0.214 0.06"/>
+        <box size="0.219 0.18 0.06"/>
       </geometry>
     </collision>

File: ijamul_description/urdf/ijamul_ros2_control.xacro (robot description, xacro)
@@ -12,5 +12,5 @@
         <hardware>
             <plugin>ijamul_firmware/ijamulInterface</plugin>
-            <param name="port">/dev/serial/by-id/usb-1a86_USB_Serial-if00-port0</param>
+            <param name="port">/dev/ttyUSB0</param>
         </hardware>
         </xacro:unless>
